File: KiCad-Shield-Uno-FlexSensor/KiCad-Shield-Uno-FlexSensor.kicad_sch (KiCad schematic)
At the start: 18 parts, among them J1 Power, J2 Digital/PWM, J3 Analog, J4 Digital/PWM, J5 Conn_01x02, U1 LTC1050

Commit message: Commencement du code pour l'arduino
Parts:
- C4: value 0,1µ -> 1µ
